Commit message: Tuned depth vision to fit test

File: src/visual/rviz/model.urdf (robot description, URDF)
Before this commit: robot arav, 2 links, 1 joints
Links:
- link robot_frame: geometry collision box size=0.47 0.47 0.11; visual mesh filename=package://visual/mesh/arav.dae scale=0.75 0.75 0.75
